Commit message: can made in blender

File: environment/can.urdf (robot description, URDF)
Before this commit: robot cola_can, 1 links, 0 joints
Links:
- link baseLink: geometry collision mesh filename=can.obj scale=0.02 0.02 0.02; visual mesh filename=can.obj scale=0.02 0.02 0.02

Commit message: improved can

File: environment/can.urdf (robot description, URDF)
Before this commit: robot cola_can, 1 links, 0 joints
Links:
- link baseLink: geometry collision mesh filename=can_decomp.obj scale=0.025 0.025 0.025; visual mesh filename=can.obj scale=1 1 1
