Commit message: pose integrated

File: simulation/room.urdf (robot description, URDF)
Before this commit: robot room.urdf, 1 links, 0 joints
Links:
- link baseLink: geometry visual mesh filename=./simulation/room.obj scale=1 1 1

File: simulation/wall.urdf (robot description, URDF)
Before this commit: robot room.urdf, 1 links, 0 joints
Links:
- link baseLink: geometry visual mesh filename=./simulation/wall.obj scale=1 1 1
