Commit message: gripping complete, pouring started

File: assets/ur5/ur5_robotiq.urdf (robot description, URDF)
Before this commit: robot ur5_robotiq, 23 links, 22 joints
Links:
- added link tool_tip_link
Joints:
- added joint tool_tip_joint: type fixed, parent ee_link, child tool_tip_link, origin xyz=0.0 0.0 0.0 rpy=0.0 0.0 0.0

File: environment/can.urdf (robot description, URDF)
Before this commit: robot can.urdf, 1 links, 0 joints
Links:
- link baseLink: mass 100 -> .5; geometry collision mesh filename=cola_can.obj; visual mesh filename=cola_can.obj

Commit message: working pour from master chef can

File: assets/ur5/ur5_robotiq.urdf (robot description, URDF)
Before this commit: robot ur5_robotiq, 24 links, 23 joints
Joints:
- joint tool_tip_joint: origin xyz=0.0 0.0 0.0 rpy=0.0 0.0 0.0 -> xyz=0.15 0.0 0.0 rpy=0.0 0.0 0.0

Commit message: completed simulation in isolation

File: assets/ur5/ur5_robotiq.urdf (robot description, URDF)
Before this commit: robot ur5_robotiq, 24 links, 23 joints
Links:
- link left_inner_finger: geometry visual mesh filename=gripper/meshes/visual/robotiq_arg2f_85_inner_finger.dae scale=0.001 0.001 0.001
- link left_inner_finger_pad: geometry visual box size=0.022 0.00635 0.0375
- link left_inner_knuckle: geometry visual mesh filename=gripper/meshes/visual/robotiq_arg2f_85_inner_knuckle.dae scale=0.001 0.001 0.001
- link left_outer_finger: geometry visual mesh filename=gripper/meshes/visual/robotiq_arg2f_85_outer_finger.dae scale=0.001 0.001 0.001
- link left_outer_knuckle: geometry visual mesh filename=gripper/meshes/visual/robotiq_arg2f_85_outer_knuckle.dae scale=0.001 0.001 0.001
- link right_inner_finger: geometry visual mesh filename=gripper/meshes/visual/robotiq_arg2f_85_inner_finger.dae scale=0.001 0.001 0.001
- link right_inner_finger_pad: geometry visual box size=0.022 0.00635 0.0375
- link right_inner_knuckle: geometry visual mesh filename=gripper/meshes/visual/robotiq_arg2f_85_inner_knuckle.dae scale=0.001 0.001 0.001
- link right_outer_finger: geometry visual mesh filename=gripper/meshes/visual/robotiq_arg2f_85_outer_finger.dae scale=0.001 0.001 0.001
- link right_outer_knuckle: geometry visual mesh filename=gripper/meshes/visual/robotiq_arg2f_85_outer_knuckle.dae scale=0.001 0.001 0.001
- link robotiq_arg2f_base_link: geometry visual mesh filename=gripper/meshes/visual/robotiq_arg2f_85_base_link.dae scale=0.001 0.001 0.001
Joints:
- joint tool_tip_joint: origin xyz=0.15 0.0 0.0 rpy=0.0 0.0 0.0 -> xyz=0.14 0.0 0.0 rpy=0.0 0.0 0.0

File: assets/ur5/ur5_robotiq_85_gripper.urdf (robot description, URDF)
Before this commit: robot assembled_robot, 21 links, 20 joints
Links:
- link robotiq_85_base_link: geometry visual mesh filename=../meshes/visual/robotiq_85_base_link.dae
- link robotiq_85_left_finger_link: geometry visual mesh filename=../meshes/visual/robotiq_85_finger_link.dae
- link robotiq_85_left_finger_tip_link: geometry visual box size=0.05 0.005 0.025
- link robotiq_85_left_inner_knuckle_link: geometry visual mesh filename=../meshes/visual/robotiq_85_inner_knuckle_link.dae
- link robotiq_85_left_knuckle_link: geometry visual mesh filename=../meshes/visual/robotiq_85_knuckle_link.dae
- link robotiq_85_right_finger_link: geometry visual mesh filename=../meshes/visual/robotiq_85_finger_link.dae
- link robotiq_85_right_finger_tip_link: geometry visual box size=0.05 0.005 0.025
- link robotiq_85_right_inner_knuckle_link: geometry visual mesh filename=../meshes/visual/robotiq_85_inner_knuckle_link.dae
- link robotiq_85_right_knuckle_link: geometry visual mesh filename=../meshes/visual/robotiq_85_knuckle_link.dae
